Commit message: add apriltags.world and change the model

File: catkin_ws/src/hector_quadrotor/hector_quadrotor_description/urdf/quadrotor_base.urdf.xacro (robot description, xacro)
@@ -25,7 +25,7 @@
     </link>
     <!-- Sonar height sensor -->
-    <xacro:sonar_sensor name="sonar" parent="base_link" ros_topic="sonar_height" update_rate="10" min_range="0.03" max_range="3.0" field_of_view="${40*pi/180}" ray_count="3">
+    <!-- <xacro:sonar_sensor name="sonar" parent="base_link" ros_topic="sonar_height" update_rate="10" min_range="0.03" max_range="3.0" field_of_view="${40*pi/180}" ray_count="3">
       <origin xyz="-0.16 0.0 -0.012" rpy="0 ${90*pi/180} 0"/>
-    </xacro:sonar_sensor>
+    </xacro:sonar_sensor> -->
   </xacro:macro>
 </robot>

File: catkin_ws/src/hector_quadrotor/hector_quadrotor_description/urdf/quadrotor_downward_cam.urdf.xacro (robot description, xacro)
@@ -1,13 +1,23 @@
 <?xml version="1.0"?>
-<robot name="quadrotor" xmlns:xacro="http://www.ros.org/wiki/xacro">
-    <xacro:property name="M_PI" value="3.1415926535897931" />
-    <!-- Included URDF Files -->
-    <xacro:include filename="$(find hector_quadrotor_description)/urdf/quadrotor_base.urdf.xacro" />
-    <!-- Instantiate quadrotor_base_macro once (has no parameters atm) -->
-    <xacro:quadrotor_base_macro />
-    <!-- Downward facing camera -->
-    <xacro:include filename="$(find hector_sensors_description)/urdf/generic_camera.urdf.xacro" />
-    <xacro:generic_camera name="downward_cam" parent="base_link" ros_topic="camera/image" cam_info_topic="camera/camera_info" update_rate="20" res_x="640" res_y="480" image_format="L8" hfov="100">
-      <origin xyz="0.4 0.0 -0.0" rpy="0 ${M_PI/2} 0"/>
-    </xacro:generic_camera>
+<robot name="quadrotor"
+  xmlns:xacro="http://www.ros.org/wiki/xacro">
+  <xacro:property name="M_PI" value="3.1415926535897931" />
+  <!-- Included URDF Files -->
+  <xacro:include filename="$(find hector_quadrotor_description)/urdf/quadrotor_base.urdf.xacro" />
+  <!-- Instantiate quadrotor_base_macro once (has no parameters atm) -->
+  <xacro:quadrotor_base_macro />
+  <!-- Downward facing camera, the unit of hfov is degree -->
+  <!-- the parameters is based on the camera of raspberry pi: SONY P5V04A -->
+  <xacro:include filename="$(find hector_sensors_description)/urdf/generic_camera.urdf.xacro" />
+  <xacro:generic_camera
+  name="downward_cam"
+  parent="base_link"
+  ros_topic="camera/image"
+  cam_info_topic="camera/camera_info"
+  update_rate="60"
+  res_x="1280" res_y="720"
+  image_format="L8"
+  hfov="65">
+    <origin xyz="0.0 0.0 -0.045" rpy="0 ${M_PI/2} 0"/>
+  </xacro:generic_camera>
 </robot>
